File: pcb/aether-l052-v1/aether-l052-v1.kicad_pcb (KiCad board)
At the start: 2 copper layers, 50.8 x 22.9 mm, 33 parts, among them J1 USB_C_Receptacle_USB2.0_16P, J2 Conn_01x16_Pin, J3 Conn_01x12_Pin, J4 Conn_01x02_Pin, J5 Conn_01x04_Pin, J6 Conn_ARM_JTAG_SWD_10, Q1 DMG2305UX-7, U1 MCP1711T-3.3I/OT, U2 MCP73831-2-OT, U3 STM32L052K8Ux

Commit message: schematic, board layout in progress
Parts:
- added C7: 10u, Capacitor_SMD:C_0805_2012Metric, F.Cu at (113.2, 92.1)
- added JP1: SolderJumper_2_Bridged, Jumper:SolderJumper-2_P1.3mm_Bridged_RoundedPad1.0x1.5mm, B.Cu at (120.5, 84.4)
- added JP2: SolderJumper_3_Bridged12, Jumper:SolderJumper-3_P1.3mm_Bridged12_RoundedPad1.0x1.5mm, B.Cu at (121.0, 88.5)
- added R8: 10k, Resistor_SMD:R_0603_1608Metric, F.Cu at (131.3, 84.7)
- added TP1: SWCLK, TestPoint:TestPoint_Pad_D2.0mm, B.Cu at (146.1, 92.7)
- added TP2: SWDIO, TestPoint:TestPoint_Pad_D2.0mm, B.Cu at (146.1, 87.6)
- J4: value Conn_01x02_Pin -> S2B-PH-SM4-TB; footprint Connector_JST:JST_PH_S2B-PH-K_1x02_P2.00mm_Horizontal -> aether-l052:S2B-PH-SM4-TB_LF__SN_
- J5: value Conn_01x04_Pin -> BM04B-SRSS-TB
- U2: value MCP73831-2-OT -> MCP73832-2-OT
- moved C5 32.2 mm to (137.4, 91.4), turned to 90 degrees
- moved R4 28.7 mm to (118.9, 91.7), turned to 90 degrees
- moved R7 28.6 mm to (109.5, 96.2), turned to -90 degrees
- moved C1 26.3 mm to (123.8, 89.5)
- moved C6 25.0 mm to (127.0, 91.5), turned to -90 degrees
- moved C4 25.0 mm to (128.4, 85.9), turned to 90 degrees
- moved D1 24.2 mm to (123.4, 95.5), turned to 180 degrees
- moved U2 23.7 mm to (116.2, 91.6), turned to -90 degrees
- moved R5 23.2 mm to (118.0, 88.5), turned to 180 degrees
- moved U1 22.5 mm to (123.9, 86.0), turned to 90 degrees
- moved R6 20.5 mm to (135.2, 84.0)
- moved R3 20.5 mm to (120.7, 96.0), turned to -90 degrees
- moved Q1 20.0 mm to (122.0, 92.6)
- moved C2 20.0 mm to (121.0, 85.6), turned to -90 degrees
- moved C3 18.2 mm to (118.2, 85.6), turned to 90 degrees
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Connections:
- net /RX renamed /A9_USART1_RX
- net /TX renamed /A10_USART1_TX
- D2 pad 2: VBUS -> Net-(D2-A)
- D3 pad 1: Net-(D3-K) -> GND
- D3 pad 2: /LED_ONBOARD -> Net-(D3-A)
- J2 pad 10: unconnected-(J2-Pin_10-Pad10) -> /A2
- J2 pad 11: unconnected-(J2-Pin_11-Pad11) -> /A1
- J2 pad 12: unconnected-(J2-Pin_12-Pad12) -> /A0
- J2 pad 4: /MISO -> /A6_SPI1_MISO
- J2 pad 5: /MOSI -> /A7_SPI1_MOSI
- J2 pad 6: /SCK -> /A5_SPI1_SCK
- J2 pad 7: unconnected-(J2-Pin_7-Pad7) -> /A8
- J2 pad 8: unconnected-(J2-Pin_8-Pad8) -> /A4_DAC
- J2 pad 9: unconnected-(J2-Pin_9-Pad9) -> /A3
- J3 pad 10: unconnected-(J3-Pin_10-Pad10) -> /B0
- J3 pad 11: /SCL -> /B6_I2C1_SCL
- J3 pad 12: /SDA -> /B7_I2C1_SDA
- J3 pad 4: unconnected-(J3-Pin_4-Pad4) -> /B8_CHRG_STAT
- J3 pad 5: unconnected-(J3-Pin_5-Pad5) -> /B5
- J3 pad 6: unconnected-(J3-Pin_6-Pad6) -> /B4
- J3 pad 7: unconnected-(J3-Pin_7-Pad7) -> /B3
- J3 pad 8: unconnected-(J3-Pin_8-Pad8) -> /B2
- J3 pad 9: unconnected-(J3-Pin_9-Pad9) -> /B1
- J5 pad MP: (no net) -> GND
- J6 pad 1: unconnected-(J6-VTref-Pad1) -> VDD
- J6 pad 10: unconnected-(J6-~{RESET}-Pad10) -> /!RESET
- J6 pad 2: unconnected-(J6-SWDIO/TMS-Pad2) -> /SWDIO
- J6 pad 3: Net-(J6-GND-Pad3) -> GND
- J6 pad 4: unconnected-(J6-SWCLK/TCK-Pad4) -> /SWCLK
- J6 pad 5: Net-(J6-GND-Pad3) -> GND
- J6 pad 9: unconnected-(J6-GNDDetect-Pad9) -> GND
- R5 pad 1: Net-(D2-K) -> Net-(JP2-C)
- R5 pad 2: Net-(U2-STAT) -> Net-(D2-A)
- R6 pad 1: Net-(D3-K) -> /A15_LED_ONBOARD
- R6 pad 2: GND -> Net-(D3-A)
- U2 pad 1: Net-(U2-STAT) -> Net-(D2-K)
- U3 pad 10: unconnected-(U3-PA4-Pad10) -> /A4_DAC
- U3 pad 11: unconnected-(U3-PA5-Pad11) -> /A5_SPI1_SCK
- U3 pad 12: unconnected-(U3-PA6-Pad12) -> /A6_SPI1_MISO
- U3 pad 13: unconnected-(U3-PA7-Pad13) -> /A7_SPI1_MOSI
- U3 pad 14: unconnected-(U3-PB0-Pad14) -> /B0
- U3 pad 15: unconnected-(U3-PB1-Pad15) -> /B1
- U3 pad 16: unconnected-(U3-PB2-Pad16) -> /B2
- U3 pad 18: unconnected-(U3-PA8-Pad18) -> /A8
- U3 pad 19: unconnected-(U3-PA9-Pad19) -> /A9_USART1_TX
- U3 pad 20: unconnected-(U3-PA10-Pad20) -> /A10_USART1_RX
- U3 pad 23: unconnected-(U3-PA13-Pad23) -> /SWDIO
- U3 pad 24: unconnected-(U3-PA14-Pad24) -> /SWCLK
- U3 pad 25: unconnected-(U3-PA15-Pad25) -> /A15_LED_ONBOARD
- U3 pad 26: unconnected-(U3-PB3-Pad26) -> /B3
- U3 pad 27: unconnected-(U3-PB4-Pad27) -> /B4
- U3 pad 28: unconnected-(U3-PB5-Pad28) -> /B5
- U3 pad 29: unconnected-(U3-PB6-Pad29) -> /B6_I2C1_SCL
- U3 pad 30: unconnected-(U3-PB7-Pad30) -> /B7_I2C1_SDA
- U3 pad 32: unconnected-(U3-PB8-Pad32) -> /B8_CHRG_STAT
- U3 pad 6: unconnected-(U3-PA0-Pad6) -> /A0
- U3 pad 7: unconnected-(U3-PA1-Pad7) -> /A1
- U3 pad 8: unconnected-(U3-PA2-Pad8) -> /A2
- U3 pad 9: unconnected-(U3-PA3-Pad9) -> /A3
Other:
- board text added: "A0"
- board text added: "A15"
- board text added: "STM32L052K8U6 64 kB flash, 8 kB RAM ultra low power battery charging"
- board text added: "SWCLK"
- board text added: "SWDIO"
- board text added: "Scl"
- board text added: "Sda"
- board text added: "github.com/xx0x/aether-l052"

Commit message: routing
Parts:
- added S2: SKRPACE010, aether-l052:SKRPACE010, F.Cu at (144.0, 95.2)
- moved TP1 5.08 mm to (146.1, 87.6)
- moved TP2 5.08 mm to (146.1, 92.7)
- moved JP2 3.17 mm to (117.8, 88.9)
- moved C5 2.34 mm to (136.7, 93.6), turned to -90 degrees
- moved J6 1.36 mm to (142.7, 88.9)
- moved R6 1.00 mm to (135.9, 84.6), turned to 90 degrees
- moved R3 0.64 mm to (120.1, 95.8), turned to 180 degrees
- moved R4 0.56 mm to (118.6, 92.2)
- moved R8 0.49 mm to (130.8, 84.7)
- moved C6 0.49 mm to (126.5, 91.4)
- moved R9 0.44 mm to (126.5, 86.3)
- moved C4 0.20 mm to (128.6, 85.9)
- moved J5 0.11 mm to (149.9, 90.2)
- moved J4 0.10 mm to (112.4, 86.5)
Connections:
- J2 pad 2: /A10_USART1_TX -> /A9_USART1_TX
- J2 pad 3: /A9_USART1_RX -> /A10_USART1_RX
- J5 pad 3: /SDA -> /B7_I2C1_SDA
- J5 pad 4: /SCL -> /B6_I2C1_SCL
Routing:
- net VDD: track 0.00 -> 106.6 mm, vias 0 -> 6
- net /!RESET: track 0.00 -> 57.8 mm, vias 0 -> 5
- net /D-: track 0.00 -> 50.3 mm, vias 0 -> 3
- net /D+: track 0.00 -> 48.1 mm, vias 0 -> 2
- net /BOOT0: track 0.00 -> 41.2 mm, vias 0 -> 2
- net Net-(D2-K): track 0.00 -> 36.9 mm, vias 0 -> 3
- net Net-(D3-A): track 0.00 -> 36.6 mm, vias 0 -> 4
- net VBUS: track 0.00 -> 35.9 mm, vias 0 -> 1
- net /B6_I2C1_SCL: track 0.00 -> 34.9 mm, vias 0 -> 2
- net /B7_I2C1_SDA: track 0.00 -> 34.0 mm, vias 0 -> 3
- net /B0: track 0.00 -> 28.5 mm, vias 0 -> 2
- net /VBAT: track 0.00 -> 27.1 mm
- net Net-(D2-A): track 0.00 -> 26.8 mm, vias 0 -> 2
- net /B1: track 0.00 -> 23.9 mm, vias 0 -> 2
- net /B2: track 0.00 -> 22.2 mm, vias 0 -> 2
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- added copper zone on B.Cu, net GND
- added copper zone on F.Cu, net GND
Other:
- board text added: "A1"
- board text added: "A2"
- board text added: "A3"
- board text added: "A4"
- board text added: "A8"
- board text added: "B0"
- board text added: "B1"
- board text added: "B2"
- board text added: "B3"
- board text added: "B4"
- board text added: "B5"
- board text added: "B8"
- board text added: "Bat"
- board text added: "Boot0"
- board text added: "Bt0"
- board text added: "Chg>B8"
- board text added: "ChgPu"
- board text added: "En"
- board text added: "Mi"
- board text added: "Mo"
- board text added: "Rx"
- board text added: "Sck"
- board text added: "Tx"
- board text added: "Usb"

Commit message: routing tweaks
Parts:
- moved S2 5.48 mm to (149.4, 94.2)
- moved J5 2.04 mm to (149.7, 88.1)
- moved J6 1.35 mm to (142.3, 90.2)
- moved U3 0.50 mm to (132.1, 90.2)
- moved C5 0.49 mm to (136.2, 93.7)
Routing:
- net /BOOT0: track 41.2 -> 49.3 mm
- net GND: track 5.72 -> 0.00 mm, vias 87 -> 94
- net VDD: track 106.6 -> 110.0 mm
- net /SWCLK: track 12.8 -> 15.8 mm
- net /B6_I2C1_SCL: track 34.9 -> 32.9 mm
- net /B7_I2C1_SDA: track 34.0 -> 32.2 mm
- net /B1: track 23.9 -> 24.8 mm
- net /!RESET: track 57.8 -> 57.0 mm
- net /SWDIO: track 13.8 -> 14.5 mm
- net /A8: track 14.5 -> 13.9 mm
- net /B2: track 22.2 -> 22.8 mm
- net /B8_CHRG_STAT: track 18.3 -> 17.7 mm
- net /B0: track 28.5 -> 29.0 mm
Other:
- board text removed: "IN PROGRESS"

Commit message: finishing board, add gerber, bom, cpl
Parts:
- J5: value BM04B-SRSS-TB -> SM04B-SRSS-TB; footprint Connector_JST:JST_SH_BM04B-SRSS-TB_1x04-1MP_P1.00mm_Vertical -> Connector_JST:JST_SH_SM04B-SRSS-TB_1x04-1MP_P1.00mm_Horizontal
- moved J5 0.71 mm to (149.0, 88.1), turned to 90 degrees
- moved J6 0.53 mm to (141.7, 90.2)
- moved C5 0.38 mm to (136.0, 94.0)
Routing:
- net /B6_I2C1_SCL: track 32.9 -> 26.6 mm
- net GND: track 0.00 -> 2.96 mm, vias 94 -> 93
- net /B7_I2C1_SDA: track 32.2 -> 29.3 mm, vias 3 -> 2
- net /SWCLK: track 15.8 -> 17.2 mm
- net /A9_USART1_TX: track 15.0 -> 14.0 mm
