File: pcb/aether-l052-v1/aether-l052-v1.kicad_sch (KiCad schematic)
At the start: 33 parts, among them J1 USB_C_Receptacle_USB2.0_16P, J2 Conn_01x16_Pin, J3 Conn_01x12_Pin, J4 Conn_01x02_Pin, J5 Conn_01x04_Pin, J6 Conn_ARM_JTAG_SWD_10, Q1 DMG2305UX-7, U1 MCP1711T-3.3I/OT, U2 MCP73831-2-OT, U3 STM32L052K8Ux

Commit message: schematic, board layout in progress
Parts:
- removed J4: Conn_01x02_Pin, Connector_JST:JST_PH_S2B-PH-K_1x02_P2.00mm_Horizontal, symbol Connector:Conn_01x02_Pin
- removed J5: Conn_01x04_Pin, Connector_JST:JST_SH_BM04B-SRSS-TB_1x04-1MP_P1.00mm_Vertical, symbol Connector:Conn_01x04_Pin
- removed U2: MCP73831-2-OT, Package_TO_SOT_SMD:SOT-23-5, symbol Battery_Management:MCP73831-2-OT
- added C7: 10u, Capacitor_SMD:C_0805_2012Metric, symbol Device:C
- added J4: S2B-PH-SM4-TB, aether-l052:S2B-PH-SM4-TB_LF__SN_, symbol aether-l052:Conn_01x02_Pin_SMD_MT
- added J5: BM04B-SRSS-TB, Connector_JST:JST_SH_BM04B-SRSS-TB_1x04-1MP_P1.00mm_Vertical, symbol aether-l052:Conn_01x04_Pin_SMD_MT
- added JP1: SolderJumper_2_Bridged, Jumper:SolderJumper-2_P1.3mm_Bridged_RoundedPad1.0x1.5mm, symbol Jumper:SolderJumper_2_Bridged
- added JP2: SolderJumper_3_Bridged12, Jumper:SolderJumper-3_P1.3mm_Bridged12_RoundedPad1.0x1.5mm, symbol Jumper:SolderJumper_3_Bridged12
- added R8: 10k, Resistor_SMD:R_0603_1608Metric, symbol Device:R
- added TP1: SWCLK, TestPoint:TestPoint_Pad_D2.0mm, symbol Connector:TestPoint
- added TP2: SWDIO, TestPoint:TestPoint_Pad_D2.0mm, symbol Connector:TestPoint
- added U2: MCP73832-2-OT, Package_TO_SOT_SMD:SOT-23-5, symbol Battery_Management:MCP73832-2-OT
Connections:
- net MISO is gone; now on net A6_SPI1_MISO: J2.4 (Pin_4)
- net MOSI is gone; now on net A7_SPI1_MOSI: J2.5 (Pin_5)
- net SCK is gone; now on net A5_SPI1_SCK: J2.6 (Pin_6)
- net !RESET: now also J6.10 (~{RESET})
- net BOOT0: now also R8.1
- net GND: now also D3.1 (K), J6.3 (GND), J6.5 (GND), J6.9 (GNDDetect), C7.2, J4.2 (Pin_2), J4.P1, J4.P2, J5.1 (Pin_1), J5.MP, R8.2, U2.2 (V_{SS}); no longer R6.2
- net SCL: now also J5.4 (Pin_4); no longer J3.11 (Pin_11)
- net SDA: now also J5.3 (Pin_3); no longer J3.12 (Pin_12)
- net VBAT: now also J4.1 (Pin_1), U2.3 (V_{BAT})
- net VBUS: now also C7.1, JP2.3 (B), U2.4 (V_{DD}); no longer D2.2 (A)
- net VDD: now also J6.1 (VTref), J5.2 (Pin_2), JP2.1 (A)
- net at R5.2: now also D2.2 (A)
- net at R4.1: now also U2.5 (PROG)
- net A4_DAC: now reaches U3.10 (PA4)
- net A4_DAC: now also J2.8 (Pin_8)
- net A5_SPI1_SCK: now reaches U3.11 (PA5)
- net A6_SPI1_MISO: now reaches U3.12 (PA6)
- net A7_SPI1_MOSI: now reaches U3.13 (PA7)
- net B0: now reaches U3.14 (PB0)
- net B0: now also J3.10 (Pin_10)
- net B1: now reaches U3.15 (PB1)
- net B1: now also J3.9 (Pin_9)
- net B2: now reaches U3.16 (PB2)
- net B2: now also J3.8 (Pin_8)
- net A8: now reaches U3.18 (PA8)
- net A8: now also J2.7 (Pin_7)
- net A9_USART1_TX: now reaches U3.19 (PA9)
- net A10_USART1_RX: now reaches U3.20 (PA10)
- net SWDIO: now reaches U3.23 (PA13)
- net SWDIO: now also J6.2 (SWDIO/TMS), TP2.1
- net SWCLK: now reaches U3.24 (PA14)
- net SWCLK: now also J6.4 (SWCLK/TCK), TP1.1
- net A15_LED_ONBOARD: now reaches U3.25 (PA15)
- net A15_LED_ONBOARD: now also R6.1
- net B3: now reaches U3.26 (PB3)
- net B3: now also J3.7 (Pin_7)
- net B4: now reaches U3.27 (PB4)
- net B4: now also J3.6 (Pin_6)
- net B5: now reaches U3.28 (PB5)
- net B5: now also J3.5 (Pin_5)
- net B6_I2C1_SCL: now reaches U3.29 (PB6)
- net B6_I2C1_SCL: now also J3.11 (Pin_11)
- net B7_I2C1_SDA: now reaches U3.30 (PB7)
- net B7_I2C1_SDA: now also J3.12 (Pin_12)
- net B8_CHRG_STAT: now reaches U3.32 (PB8)
- net B8_CHRG_STAT: now also J3.4 (Pin_4), JP1.2 (B)
- net A0: now reaches U3.6 (PA0)
- net A0: now also J2.12 (Pin_12)
- net A1: now reaches U3.7 (PA1)
- net A1: now also J2.11 (Pin_11)
- net A2: now reaches U3.8 (PA2)
- net A2: now also J2.10 (Pin_10)
- net A3: now reaches U3.9 (PA3)
- net A3: now also J2.9 (Pin_9)
- net at D2.1 (K): now also JP1.1 (A), U2.1 (STAT); no longer R5.1
- net LED_ONBOARD: no longer names the net of D3.2 (A)
- net LED_ONBOARD: now also R6.2
- net RX renamed A9_USART1_RX
- net TX renamed A10_USART1_TX
- new net: JP2.2 (C), R5.1
Other:
- note added: "10k = approx 100mA charge current LED uses VDD so we can sense it using MCU"
- note added: "PA0 = WKUP1"
- note removed: "10k approx 100mA charge current"
- moved on the sheet: D2, D3, H1, H2, H3, H4, J2, J6, R5, R6, U3

Commit message: routing
Parts:
- added S2: SKRPACE010, aether-l052:SKRPACE010, symbol aether-l052:SKRPACE010
Connections:
- net A10_USART1_TX is gone; now on net A9_USART1_TX: J2.2 (Pin_2)
- net A9_USART1_RX is gone; now on net A10_USART1_RX: J2.3 (Pin_3)
- net SCL is gone; now on net B6_I2C1_SCL: J5.4 (Pin_4)
- net SDA is gone; now on net B7_I2C1_SDA: J5.3 (Pin_3)
- net BOOT0: now also S2.3, S2.4
- net VDD: now also S2.1, S2.2
Other:
- note added: "Chg>B8"
- note added: "ChgPu"
- moved on the sheet: R8

Commit message: routing tweaks
Other:
- note removed: "IN PROGRESS"
Changed lines of the file:
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@@
 		(rev "1")
 		(company "github.com/xx0x/aether-l052")
-		(comment 1 "A dev board based on STM32L052K8U6")
+		(comment 1 "License: CERN-OHL-P-2.0")
 		(comment 2 "Ultra-low standby mode, battery charger")
+		(comment 3 "A dev board based on STM32L052K8U6")
 	)
 	(text "150mA\nultra low quiescent current"
@@
 			)
 		)
-	)
-	(text "IN PROGRESS"
-		(exclude_from_sim no)
-		(at 218.948 143.764 0)
-		(effects
-			(font
-				(size 10.16 10.16)
-				(thickness 1.524)
-				(bold yes)
-			)
-		)

Commit message: finishing board, add gerber, bom, cpl
Parts:
- C1, C2, C3, C7: LCSC (none) -> C15850
- C4, C5, C6: LCSC (none) -> C14663
- D1: LCSC (none) -> C7380001
- D2: LCSC (none) -> C2286
- D3: LCSC (none) -> C2290
- F1: LCSC (none) -> C883109
- J1: LCSC (none) -> C393939
- J4: LCSC (none) -> C295747
- J5: value BM04B-SRSS-TB -> SM04B-SRSS-TB; footprint Connector_JST:JST_SH_BM04B-SRSS-TB_1x04-1MP_P1.00mm_Vertical -> Connector_JST:JST_SH_SM04B-SRSS-TB_1x04-1MP_P1.00mm_Horizontal; LCSC (none) -> C160404
- J6: LCSC (none) -> C41376037
- Q1: LCSC (none) -> C150470
- R1, R2: LCSC (none) -> C23186
- R3, R4, R7, R8, R9: LCSC (none) -> C25804
- R5, R6: LCSC (none) -> C21190
- S1, S2: LCSC (none) -> C139797
- U1: LCSC (none) -> C79527
- U2: LCSC (none) -> C38066
- U3: LCSC (none) -> C1342049
